File: pcb/selflace.brd (EAGLE design)
At the start: 25.4 x 47 mm, 41 parts, among them IC1 78L05Z, J3 AVR_SPI_PROG_3X2NS, U1 ATMEGA328P_TQFP, Y1 16MHz

Commit message: routing is hell and i hate it
Parts:
- removed C1, C11: 0.1uF, SparkFun-Capacitors:0603
- removed C10, C5: 1.0uF, SparkFun-Capacitors:0603
- added D1, D2, D3, D4: (no value), SparkFun-LED:LED-1206
- added R10, R11, R8, R9: 220, SparkFun-Resistors:0603
- Y1: device SparkFun-Clocks:HC49US -> SparkFun-Clocks:CRYSTAL-SMD-5X3.2-4PAD
- moved Y1 3.45 mm to (9.40, 44.2), turned to 180 degrees
Connections:
- new net N$14: D1.A, R8.2
- new net N$15: D2.A, R9.2
- new net N$16: D3.A, R10.2
- new net N$17: D4.A, R11.2
- net DIG2: now also R8.1
- net DIG3: now also R9.1
- net DIG8: now also R10.1
- net DIG9: now also R11.1
- net GND: now also D1.C, D2.C, D3.C, D4.C; no longer C1.2, C10.2, C11.2, C5.2
- net N$7: now also Y1.3; no longer Y1.2
- net VCC: no longer C1.1, C10.1, C11.1, C5.1
Routing:
- net GND: track 174.1 -> 0.00 mm, vias 1 -> 0
- net MISO: track 90.5 -> 0.00 mm, vias 2 -> 0
- net MOSI: track 64.1 -> 0.00 mm, vias 5 -> 0
- net VCC: track 154.2 -> 97.6 mm, vias 3 -> 4
- net N$7: track 55.6 -> 0.00 mm, vias 1 -> 0
- net N$2: track 49.1 -> 0.00 mm, vias 2 -> 0
- net N$11: track 42.0 -> 0.00 mm, vias 3 -> 0
- net SCK: track 33.3 -> 0.00 mm, vias 1 -> 0
- net RESET: track 32.7 -> 0.00 mm
- net N$1: track 30.6 -> 0.00 mm, vias 2 -> 0
- net N$5: track 23.7 -> 0.00 mm, vias 2 -> 0
- net N$9: track 22.3 -> 0.00 mm, vias 3 -> 0
- net N$4: track 21.0 -> 0.00 mm
- net N$10: track 18.6 -> 0.00 mm, vias 1 -> 0
- net N$6: track 17.2 -> 0.00 mm, vias 1 -> 0
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Other:
- board text added: "BKW"
- board text added: "FWD"
- board text added: "ON"
- board text added: "STAT"

Commit message: yay, it's a thing that does a thing that's made to do a thing
Routing:
- net N$11: track 0.00 -> 64.9 mm, vias 0 -> 5
- net N$2: track 0.00 -> 61.2 mm, vias 0 -> 4
- net N$7: track 0.00 -> 52.5 mm, vias 0 -> 6
- net RESET: track 0.00 -> 40.2 mm, vias 0 -> 3
- net DIG3: track 0.00 -> 37.1 mm, vias 0 -> 2
- net N$1: track 0.00 -> 37.0 mm, vias 0 -> 2
- net MOSI: track 0.00 -> 36.7 mm, vias 0 -> 1
- net DIG9: track 0.00 -> 35.3 mm, vias 0 -> 2
- net MISO: track 0.00 -> 33.4 mm, vias 0 -> 1
- net SCK: track 0.00 -> 32.8 mm, vias 0 -> 3
- net DIG2: track 0.00 -> 32.7 mm, vias 0 -> 2
- net N$6: track 0.00 -> 32.2 mm
- net N$9: track 0.00 -> 32.0 mm, vias 0 -> 2
- net N$4: track 0.00 -> 31.6 mm, vias 0 -> 1
- net DIG8: track 0.00 -> 26.0 mm, vias 0 -> 2
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- added copper zone on layer 1, net GND
- added copper zone on layer 16, net GND
